File: kicad/jomac-comando-mach-3.sch (KiCad schematic (older format))
At the start: 80 parts, among them Q1 Q_NPN_CBE, Q10 PN4917, Q2 C, Q3 Q_NPN_CBE, Q4 Q_NPN_CBE, Q5 Q_NPN_CBE, Q6 Q_NPN_CBE, Q7 Q_NPN_CBE, Q8 MPS3646, Q9 MPS3646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

Commit message: Fix ST-trim pin 3 not being actually connected.
Convert to KiCAD 4.05 file format
Parts:
- BT1: symbol Battery -> Battery-RESCUE-jomac-comando-mach-3
- D5: symbol LED -> LED-RESCUE-jomac-comando-mach-3
- RV1, RV2, RV3, RV4, RV5: symbol POT -> POT-RESCUE-jomac-comando-mach-3
Connections:
- net at R14.1, RV4.2: no longer RV4.3
Other:
- moved on the sheet: RV4
